File: ETL_full_module_wirebonding_mock_top/ETL_full_module_wirebonding_mock_top.kicad_pcb (KiCad board)
At the start: 2 copper layers, 47.6 x 42.6 mm, 8 parts

Commit message: Updates ETL_full_module_wirebonding_mock_base and top
Parts:
- removed the ETROC** at (46.6, 6.00)
- removed the ETROC** at (46.6, 36.6)
- removed the REF** at (5.00, 37.6)
- removed the REF** at (5.00, 5.00)
- removed the REF** at (42.6, 6.00)
- added REF**: crossed_circle_fiducial, unl_silab:crossed_circle_fiducial, F.Cu at (2.00, 39.7)
- added REF**: crossed_circle_fiducial, unl_silab:crossed_circle_fiducial, F.Cu at (2.00, 2.00)
- added REF**: crossed_circle_fiducial, unl_silab:crossed_circle_fiducial, F.Cu at (20.3, 2.00)
- moved REF** 22.4 mm to (20.3, 39.7)
- moved ETROC** 0.45 mm to (1.00, 36.1)
- moved ETROC** 0.45 mm to (1.00, 5.55)
Other:
- board size 47.6 x 42.6 mm -> 22.3 x 41.7 mm
