File: ETL/etl_etroc_mockup_v1p1/etl_etroc_mockup_v1p1.kicad_pcb (KiCad board)
At the start: 2 copper layers, 21 x 23 mm, 4 parts

Commit message: Adds work over last few months :o
Other:
- net class Default removed
