File: ETL/etl_lgad_mockup_v1p1/etl_lgad_mockup_v1p1.kicad_pcb (KiCad board)
At the start: 2 copper layers, 21.6 x 21.4 mm, 4 parts

Commit message: Adds work over last few months :o
Other:
- net class Default removed
