File: ETL/etl_module_pcb_mockup_v3p2/etl_module_pcb_mockup_v3p2.kicad_pcb (KiCad board)
At the start: 2 copper layers, 43.1 x 57.5 mm, 16 parts, among them J1 WP7B-S050VA1-R8000, J2 WP7B-S050VA1-R8000

Commit message: Adds work over last few months :o
Other:
- net class Default removed
