File: ETL/etl_module_pcb_thermal_mockup_v3/etl_module_pcb_thermal_mockup_v3.kicad_pcb (KiCad board)
At the start: 4 copper layers, 44.1 x 57.5 mm, 33 parts, among them J3 Conn_02x05_Counter_Clockwise, U1 ETROC_dummy_thermal_sensors, U2 ETROC_dummy_thermal_sensors, U3 ETROC_dummy_thermal_sensors, U4 ETROC_dummy_thermal_sensors, U5 AD77x8, U6 AD780, Y1 32kHz

Commit message: more routing
Routing:
- net /V_{ref}: track 0.00 -> 16.7 mm
- net +5V: track 17.4 -> 30.8 mm, vias 10 -> 13
- net /ETROC3: track 7.36 -> 18.6 mm
- net GND: track 29.9 -> 39.7 mm, vias 19 -> 21
- net /LGAD3: track 8.82 -> 14.3 mm
Changed lines of the file:
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@@
   (segment (start 42.8 32.5) (end 39.1 28.8) (width 0.127) (layer "B.Cu") (net 1))
   (segment (start 42.8 52.5) (end 42.8 32.5) (width 0.127) (layer "B.Cu") (net 1))
+  (segment (start 18.2 13) (end 18.2 13.05) (width 0.127) (layer "F.Cu") (net 2))
   (via (at 27.25 28.7) (size 0.4573) (drill 0.254) (layers "F.Cu" "B.Cu") (net 2))
+  (via (at 7.3 28.75) (size 0.4573) (drill 0.254) (layers "F.Cu" "B.Cu") (net 2))
   (via (at 37.3 56.3) (size 0.4573) (drill 0.254) (layers "F.Cu" "B.Cu") (net 2))
   (via (at 7.8 56) (size 0.4573) (drill 0.254) (layers "F.Cu" "B.Cu") (net 2))
+  (via (at 18.2 13.05) (size 0.4573) (drill 0.254) (layers "F.Cu" "B.Cu") (net 2))
+  (via (at 14.25 2.8) (size 0.4573) (drill 0.254) (layers "F.Cu" "B.Cu") (net 2))
   (via (at 13.5 56) (size 0.4573) (drill 0.254) (layers "F.Cu" "B.Cu") (net 2))
   (via (at 33 56.3) (size 0.4573) (drill 0.254) (layers "F.Cu" "B.Cu") (net 2))
+  (via (at 2.05 13.05) (size 0.4573) (drill 0.254) (layers "F.Cu" "B.Cu") (net 2))
   (via (at 8 2.1) (size 0.4573) (drill 0.254) (layers "F.Cu" "B.Cu") (net 2))
   (via (at 39.8 13.05) (size 0.4573) (drill 0.254) (layers "F.Cu" "B.Cu") (net 2))
   (via (at 14.2 4.2) (size 0.4573) (drill 0.254) (layers "F.Cu" "B.Cu") (net 2))
-  (via (at 12 2.1) (size 0.4573) (drill 0.254) (layers "F.Cu" "B.Cu") (net 2))
   (via (at 9 3.8) (size 0.4573) (drill 0.254) (layers "F.Cu" "B.Cu") (net 2))
   (segment (start 13.8375 4.2) (end 14.2 4.2) (width 0.127) (layer "B.Cu") (net 2))
@@
   (segment (start 36 56) (end 36.3 56.3) (width 0.127) (layer "B.Cu") (net 2))
   (segment (start 41 14.9625) (end 41 14.25) (width 0.127) (layer "B.Cu") (net 2))
+  (segment (start 13.55 2.1) (end 14.25 2.8) (width 0.127) (layer "B.Cu") (net 2))
   (segment (start 32 56) (end 32.7 56) (width 0.127) (layer "B.Cu") (net 2))
-  (segment (start 13 2.1) (end 12 2.1) (width 0.127) (layer "B.Cu") (net 2))
+  (segment (start 6 33) (end 7.3 31.7) (width 0.127) (layer "B.Cu") (net 2))
+  (segment (start 3.815 11.285) (end 2.05 13.05) (width 0.127) (layer "B.Cu") (net 2))
+  (segment (start 7.3 31.7) (end 7.3 28.75) (width 0.127) (layer "B.Cu") (net 2))
+  (segment (start 5.36 11.285) (end 3.815 11.285) (width 0.127) (layer "B.Cu") (net 2))
+  (segment (start 16.485 11.285) (end 18.2 13) (width 0.127) (layer "B.Cu") (net 2))
   (segment (start 13.0375 5) (end 13.8375 4.2) (width 0.127) (layer "B.Cu") (net 2))
   (segment (start 38.035 14.605) (end 40.6425 14.605) (width 0.127) (layer "B.Cu") (net 2))
   (segment (start 8.975329 5) (end 9 4.975329) (width 0.127) (layer "B.Cu") (net 2))
+  (segment (start 13 2.1) (end 13.55 2.1) (width 0.127) (layer "B.Cu") (net 2))
   (segment (start 9 2.1) (end 8 2.1) (width 0.127) (layer "B.Cu") (net 2))
   (segment (start 24.575 28.75) (end 27.2 28.75) (width 0.127) (layer "B.Cu") (net 2))
@@
   (segment (start 41 14.25) (end 39.8 13.05) (width 0.127) (layer "B.Cu") (net 2))
   (segment (start 36.3 56.3) (end 37.3 56.3) (width 0.127) (layer "B.Cu") (net 2))
+  (segment (start 14.96 11.285) (end 16.485 11.285) (width 0.127) (layer "B.Cu") (net 2))
   (segment (start 27.2 28.75) (end 27.25 28.7) (width 0.127) (layer "B.Cu") (net 2))
   (segment (start 40.6425 14.605) (end 41 14.9625) (width 0.127) (layer "B.Cu") (net 2))
@@
   (segment (start 4.129671 53.331873) (end 4.129671 52.829671) (width 0.127) (layer "F.Cu") (net 11))
   (segment (start 4.129671 52.829671) (end 4 52.7) (width 0.127) (layer "F.Cu") (net 11))
+  (via (at 3.35 28.75) (size 0.4573) (drill 0.254) (layers "F.Cu" "B.Cu") (net 11))
   (via (at 19.05 36.75) (size 0.4573) (drill 0.254) (layers "F.Cu" "B.Cu") (net 11))
   (via (at 4 52.7) (size 0.4573) (drill 0.254) (layers "F.Cu" "B.Cu") (net 11))
@@
   (via (at 41.35 13.05) (size 0.4573) (drill 0.254) (layers "F.Cu" "B.Cu") (net 11))
   (via (at 5.5 52.9) (size 0.4573) (drill 0.254) (layers "F.Cu" "B.Cu") (net 11))
+  (via (at 1.9 20.85) (size 0.4573) (drill 0.254) (layers "F.Cu" "B.Cu") (net 11))
   (via (at 13.75 28.65) (size 0.4573) (drill 0.254) (layers "F.Cu" "B.Cu") (net 11))
   (via (at 13.1 28.65) (size 0.4573) (drill 0.254) (layers "F.Cu" "B.Cu") (net 11))
@@
   (segment (start 41 17.0375) (end 41.2625 17.0375) (width 0.127) (layer "B.Cu") (net 11))
   (segment (start 39.7 20.55) (end 40 20.85) (width 0.127) (layer "B.Cu") (net 11))
+  (segment (start 14.96 28.04) (end 14.35 28.65) (width 0.127) (layer "B.Cu") (net 11))
   (segment (start 15.405 13) (end 17 13) (width 0.127) (layer "B.Cu") (net 11))
   (segment (start 5.36 12.555) (end 4.856571 13.058429) (width 0.127) (layer "B.Cu") (net 11))
   (segment (start 10.9625 5) (end 11 4.9625) (width 0.127) (layer "B.Cu") (net 11))
+  (segment (start 3.015 22.715) (end 1.9 21.6) (width 0.127) (layer "B.Cu") (net 11))
+  (segment (start 4 30) (end 3.35 29.35) (width 0.127) (layer "B.Cu") (net 11))
   (segment (start 38.035 17.145) (end 40.8925 17.145) (width 0.127) (layer "B.Cu") (net 11))
   (segment (start 4.856571 13.058429) (end 3.076505 13.058429) (width 0.127) (layer "B.Cu") (net 11))
   (segment (start 18.5 36.75) (end 19.05 36.75) (width 0.4) (layer "B.Cu") (net 11))
+  (segment (start 14.96 25.255) (end 14.96 28.04) (width 0.127) (layer "B.Cu") (net 11))
   (segment (start 19.525 33.83) (end 19.525 35.725) (width 0.5) (layer "B.Cu") (net 11))
   (segment (start 6.900329 5) (end 7.1 5) (width 0.127) (layer "B.Cu") (net 11))
   (segment (start 11.95 28.7) (end 13.05 28.7) (width 0.3) (layer "B.Cu") (net 11))
   (segment (start 19.525 35.725) (end 18.5 36.75) (width 0.5) (layer "B.Cu") (net 11))
+  (segment (start 3.35 29.35) (end 3.35 28.75) (width 0.127) (layer "B.Cu") (net 11))
   (segment (start 42.05 16.25) (end 42.05 13.75) (width 0.127) (layer "B.Cu") (net 11))
   (segment (start 14.35 28.65) (end 13.75 28.65) (width 0.3) (layer "B.Cu") (net 11))
   (segment (start 14.96 12.555) (end 15.405 13) (width 0.127) (layer "B.Cu") (net 11))
   (segment (start 14.96 13.445) (end 15.405 13) (width 0.127) (layer "B.Cu") (net 11))
+  (segment (start 1.9 21.6) (end 1.9 20.85) (width 0.127) (layer "B.Cu") (net 11))
   (segment (start 38.75 20.55) (end 39.7 20.55) (width 0.127) (layer "B.Cu") (net 11))
+  (segment (start 5.36 22.715) (end 3.015 22.715) (width 0.127) (layer "B.Cu") (net 11))
   (segment (start 7.1 5) (end 7.9 4.2) (width 0.127) (layer "B.Cu") (net 11))
   (segment (start 11 4.9625) (end 11 3.8) (width 0.127) (layer "B.Cu") (net 11))
@@
   (segment (start 1.4 41.3) (end 9.95 32.75) (width 0.3) (layer "B.Cu") (net 12))
   (segment (start 1.4 51.55) (end 1.4 50.8) (width 0.3) (layer "B.Cu") (net 12))
+  (segment (start 11.685 22.715) (end 14.96 22.715) (width 0.127) (layer "B.Cu") (net 13))
+  (segment (start 6 30) (end 6 28.4) (width 0.127) (layer "B.Cu") (net 13))
+  (segment (start 4 32) (end 4 33) (width 0.127) (layer "B.Cu") (net 13))
+  (segment (start 6 28.4) (end 11.685 22.715) (width 0.127) (layer "B.Cu") (net 13))
+  (segment (start 6 30) (end 4 32) (width 0.127) (layer "B.Cu") (net 13))
   (segment (start 18.715671 53.331873) (end 18.715671 52.915671) (width 0.127) (layer "F.Cu") (net 14))
   (segment (start 18.715671 52.915671) (end 18.6 52.8) (width 0.127) (layer "F.Cu") (net 14))
@@
   (segment (start 3.8 4.6) (end 3.719329 4.519329) (width 0.127) (layer "F.Cu") (net 41))
   (via (at 4.4 4.2) (size 0.4573) (drill 0.254) (layers "F.Cu" "B.Cu") (net 41))
+  (segment (start 11 2.1) (end 11.9 3) (width 0.127) (layer "B.Cu") (net 41))
   (segment (start 9.8 3.3) (end 5.3 3.3) (width 0.127) (layer "B.Cu") (net 41))
+  (segment (start 11.9 7.05) (end 11.8 7.15) (width 0.127) (layer "B.Cu") (net 41))
+  (segment (start 11.9 3) (end 11.9 7.05) (width 0.127) (layer "B.Cu") (net 41))
   (segment (start 5.3 3.3) (end 4.4 4.2) (width 0.127) (layer "B.Cu") (net 41))
   (segment (start 11 2.1) (end 9.8 3.3) (width 0.127) (layer "B.Cu") (net 41))
@@
   (segment (start 1.717329 3.517329) (end 1.717329 4.168127) (width 0.127) (layer "F.Cu") (net 42))
   (via (at 1.5 3.3) (size 0.4573) (drill 0.254) (layers "F.Cu" "B.Cu") (net 42))
+  (segment (start 8 1.1) (end 11.6 1.1) (width 0.127) (layer "B.Cu") (net 42))
   (segment (start 2.1 3) (end 1.8 3) (width 0.127) (layer "B.Cu") (net 42))
   (segment (start 6.1 3) (end 2.1 3) (width 0.127) (layer "B.Cu") (net 42))
+  (segment (start 11.6 1.1) (end 12.2095 1.7095) (width 0.127) (layer "B.Cu") (net 42))
+  (segment (start 12.2095 1.7095) (end 12.2095 7.0405) (width 0.127) (layer "B.Cu") (net 42))
+  (segment (start 7 2.1) (end 8 1.1) (width 0.127) (layer "B.Cu") (net 42))
+  (segment (start 12.2095 7.0405) (end 12.2 7.05) (width 0.127) (layer "B.Cu") (net 42))
   (segment (start 7 2.1) (end 6.1 3) (width 0.127) (layer "B.Cu") (net 42))
   (segment (start 1.8 3) (end 1.5 3.3) (width 0.127) (layer "B.Cu") (net 42))

Commit message: Finishes layout
Parts:
- added 2.5V: TestPoint, TestPoint:TestPoint_Pad_1.0x1.0mm, B.Cu at (29.4, 17.1)
- added 5V: TestPoint, TestPoint:TestPoint_Pad_1.0x1.0mm, B.Cu at (16.0, 31.3)
- added E1: TestPoint, TestPoint:TestPoint_Pad_1.0x1.0mm, B.Cu at (19.5, 56.0)
- added E2: TestPoint, TestPoint:TestPoint_Pad_1.0x1.0mm, B.Cu at (26.6, 56.0)
- added E3: TestPoint, TestPoint:TestPoint_Pad_1.0x1.0mm, B.Cu at (17.7, 1.70)
- added E4: TestPoint, TestPoint:TestPoint_Pad_1.0x1.0mm, B.Cu at (24.5, 1.70)
- added G***: LOGO, unl_silab:NLOGO, B.Cu at (41.6, 48.5)
- added GND: TestPoint, TestPoint:TestPoint_Pad_1.0x1.0mm, B.Cu at (16.0, 33.3)
- added L1: TestPoint, TestPoint:TestPoint_Pad_1.0x1.0mm, B.Cu at (17.6, 56.0)
- added L2: TestPoint, TestPoint:TestPoint_Pad_1.0x1.0mm, B.Cu at (24.8, 56.0)
- added L3: TestPoint, TestPoint:TestPoint_Pad_1.0x1.0mm, B.Cu at (19.6, 1.70)
- added L4: TestPoint, TestPoint:TestPoint_Pad_1.0x1.0mm, B.Cu at (26.6, 1.70)
- added VCC: TestPoint, TestPoint:TestPoint_Pad_1.0x1.0mm, B.Cu at (31.8, 28.9)
- added V_{ref}: TestPoint, TestPoint:TestPoint_Pad_1.0x1.0mm, B.Cu at (4.45, 34.9)
Connections:
- J3 pad 5: +5V -> VCC
- J3 pad 6: VCC -> +5V
- U5 pad 1: /ETROC4 -> /LGAD4
- U5 pad 11: /ETROC3 -> /ETROC2
- U5 pad 2: /LGAD4 -> /ETROC4
- U5 pad 7: /ETROC1 -> /ETROC3
- U5 pad 9: /ETROC2 -> /ETROC1
Routing:
- net VCC: track 91.3 -> 150.3 mm, vias 2 -> 5
- net /LGAD3: track 14.3 -> 54.1 mm, vias 1 -> 3
- net /LGAD4: track 0.00 -> 37.9 mm, vias 0 -> 2
- net /ETROC3: track 18.6 -> 48.9 mm, vias 1 -> 3
- net /ETROC4: track 0.00 -> 28.6 mm, vias 0 -> 2
- net /LGAD1: track 48.6 -> 69.0 mm, vias 2 -> 3
- net /ETROC2: track 62.4 -> 76.2 mm, vias 2 -> 3
- net /LGAD2: track 62.5 -> 75.0 mm, vias 2 -> 3
- net /V_{ref}: track 16.7 -> 28.5 mm
- net GND: track 39.7 -> 48.8 mm, vias 21 -> 26
- net /ETROC1: track 44.9 -> 53.7 mm, vias 2 -> 3
- net +5V: track 30.8 -> 36.0 mm, vias 13 -> 17
- net /2.5V: track 37.9 -> 41.5 mm
- net /~{RDY}: track 29.1 -> 31.1 mm
- net /VSS: track 103.4 -> 105.2 mm
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Other:
- board text added: "1"
- board text added: "2"
- board text added: "3"
- board text added: "4"
- board text added: "CS ~{RST} ~{RDY} NC VCC +5V DIN DOUT CLK GND"
- board text added: "Channels: 1: ETROC3 2: LGAD1 3: ETROC1 4: LGAD2 5: ETROC2 6: LGAD3 7: LGAD4 8: ETROC4"
- board text added: "Chip Numbering"
- board text added: "ETL Module PCB Thermal Mockup V3 C. Fangmeier 03-2023"
- board text added: "Fill JMPR1 for PCB heating Fill JMPR2 for chip heating"
- board text added: "Populate for 2.5V on REFIN2"
- board text removed: "CS ~{RST} ~{RDY} NC +5V VCC DOUT DIN CLK GND"
- board text removed: "Populate JMPR1 for PCB heating Populate JMPR2 for chip heating"
