File: ETL/etl_module_pcb_thermal_mockup_v3/etl_module_pcb_thermal_mockup_v3.kicad_pcb (KiCad board)
At the start: 4 copper layers, 44.1 x 57.5 mm, 47 parts, among them J3 Conn_02x05_Counter_Clockwise, U1 ETROC_dummy_thermal_sensors, U2 ETROC_dummy_thermal_sensors, U3 ETROC_dummy_thermal_sensors, U4 ETROC_dummy_thermal_sensors, U5 AD77x8, U6 AD780, Y1 32kHz

Commit message: tweaks
Parts:
- moved Y1 0.40 mm to (2.40, 9.40)
Routing:
- net Net-(JMPR1-Pad1): track 26.4 -> 28.6 mm, vias 2 -> 4
- net VCC: track 150.3 -> 151.7 mm
- net /LGAD4: track 37.9 -> 38.4 mm

Commit message: Adds firmware and wirebonding instructions to ETL thermal mockup
Parts:
- moved G*** 1.00 mm to (41.7, 49.5)
Other:
- board text added: "ETL Module PCB Thermal Mockup V3 C. Fangmeier 03-2023 https://tinyurl.com/hdvt5jh5"
- board text removed: "ETL Module PCB Thermal Mockup V3 C. Fangmeier 03-2023"
